Commit message: Enhance UAV camera handling with non-static model for attached-camera teleport spawns

File: src/lrs_halmstad/xacro/lrs_m100_base.sdf.xacro (robot description, xacro)
@@ -1,5 +1,5 @@
 <?xml version="1.0" encoding="UTF-8"?>
 <robot xmlns:xacro="http://www.ros.org/wiki/xacro">
-  <xacro:macro name="lrs_m100_macro" params="base_link_name">
+  <xacro:macro name="lrs_m100_macro" params="base_link_name base_link_kinematic:=false">
 <frame name="lidar_frame" attached_to="${base_link_name}">
     <pose>0.0 0 0.5 0 0 0</pose>
@@ -7,4 +7,6 @@
       <link name="${base_link_name}">
              <pose rotation_format="euler_rpy" degrees="true">0 0 0 0 0 0</pose>
+            <gravity>false</gravity>
+            <kinematic>${base_link_kinematic}</kinematic>
             <visual name="visual">
                 <pose>0 0 0 0 0 0</pose>

File: src/lrs_halmstad/xacro/lrs_model.xacro (robot description, xacro)
@@ -3,4 +3,5 @@
   <xacro:arg name="name" default="dji0"/>
   <xacro:arg name="model_static" default="false"/>
+  <xacro:arg name="base_link_kinematic" default="false"/>
   <model name="$(arg name)">
     <static>$(arg model_static)</static>
@@ -77,9 +78,11 @@
     <xacro:if value="${prop_type == 'm100'}">
       <xacro:include filename="$(find lrs_halmstad)/xacro/lrs_m100_base.sdf.xacro"/>
-      <xacro:lrs_m100_macro base_link_name="$(arg base_link_frame)"/>
+      <xacro:lrs_m100_macro base_link_name="$(arg base_link_frame)"
+                            base_link_kinematic="$(arg base_link_kinematic)"/>
     </xacro:if>
     <xacro:if value="${prop_type == 'm300'}">
       <xacro:include filename="$(find lrs_halmstad)/xacro/lrs_m100_base.sdf.xacro"/>
-      <xacro:lrs_m100_macro base_link_name="$(arg base_link_frame)"/>
+      <xacro:lrs_m100_macro base_link_name="$(arg base_link_frame)"
+                            base_link_kinematic="$(arg base_link_kinematic)"/>
     </xacro:if>
     <!--link name="world"/-->
@@ -132,6 +135,4 @@
             <xyz>0 0 1</xyz>
             <limit>
-              <lower>-3.1416</lower>
-              <upper>3.1416</upper>
               <effort>100</effort>
               <velocity>-1</velocity>
