Commit message: Update Baylands navigation configurations and lidar settings

File: src/lrs_halmstad/clearpath/lidar3d_0_override.urdf.xacro (robot description, xacro)
@@ -7,13 +7,13 @@
   <xacro:velodyne_lidar
       name="lidar3d_0"
-      parent_link="default_mount"
-      ang_res_h="0.4"
+      parent_link="sensor_arch_mount"
+      ang_res_h="0.5"
       ang_res_v="2.0"
       min_ang_h="-3.141592"
       max_ang_h="3.141592"
-      min_ang_v="-0.261799"
-      max_ang_v="0.261799"
-      min_range="0.5"
-      max_range="50.0"
+      min_ang_v="-0.35"
+      max_ang_v="0.4"
+      min_range="0.45"
+      max_range="25.0"
       update_rate="10">
     <origin xyz="0.0 0.0 0.0" rpy="0.0 0.0 0.0"/>

File: src/lrs_halmstad/clearpath/robot.urdf.xacro (robot description, xacro)
@@ -19,16 +19,15 @@
     <origin xyz="0.0 0.0 0.0" rpy="0.0 0.0 0.0"/>
   </xacro:top_plate>
+  <xacro:include filename="$(find clearpath_platform_description)/urdf/a200/attachments/sensor_arch.urdf.xacro"/>
+  <xacro:sensor_arch name="sensor_arch" model="sensor_arch_300" parent_link="default_mount">
+    <origin xyz="0.0 0.0 0.0" rpy="0.0 0.0 0.0"/>
+  </xacro:sensor_arch>
   <!-- Links -->
   <!-- Mounts -->
   <!-- Sensors -->
-  <!-- lidar2d_0 -->
-  <xacro:include filename="$(find clearpath_sensors_description)/urdf/hokuyo_ust.urdf.xacro"/>
-  <xacro:hokuyo_ust name="lidar2d_0" parent_link="base_link" ang_res="0.5" min_ang="-3.141592653589793" max_ang="3.141592653589793" min_range="0.05" max_range="25.0" update_rate="40">
-    <origin xyz="0.21 0.13 0.2" rpy="0.0 0.0 0.0"/>
-  </xacro:hokuyo_ust>
   <!-- camera_0 -->
   <xacro:include filename="$(find clearpath_sensors_description)/urdf/intel_realsense.urdf.xacro"/>
   <xacro:intel_realsense name="camera_0" parent_link="base_link" update_rate="30" image_height="480" image_width="640" model="d435">
-    <origin xyz="0.31 0.0 0.23" rpy="0.0 0.0 0.0"/>
+    <origin xyz="0.31 0.0 0.18" rpy="0.0 -0.1 0.0"/>
   </xacro:intel_realsense>
   <!-- Manipulators -->
