Commit message: Add RViz configuration files for follow and localization testing

File: src/lrs_halmstad/clearpath/robot.urdf.xacro (robot description, xacro)
@@ -28,6 +28,6 @@
   <!-- camera_0 -->
   <xacro:include filename="$(find clearpath_sensors_description)/urdf/intel_realsense.urdf.xacro"/>
-  <xacro:intel_realsense name="camera_0" parent_link="base_link" update_rate="30" image_height="480" image_width="640" model="d435">
-    <origin xyz="0.31 0.0 0.18" rpy="0.0 -0.1 0.0"/>
+  <xacro:intel_realsense name="camera_0" parent_link="base_link" update_rate="20" image_height="480" image_width="640" model="d435">
+    <origin xyz="0.36 0.0 0.15" rpy="0.0 -0.2 0.0"/>
   </xacro:intel_realsense>
   <!-- Manipulators -->
